File: Chromatic/Chromatic.kicad_sch (KiCad schematic)
At the start: 110 parts, among them SW1 SW_DPST_x2, SW10 SW_DPST_x2, SW100 SW_DPST_x2, SW101 SW_DPST_x2, SW102 SW_DPST_x2, SW103 SW_DPST_x2, SW104 SW_DPST_x2, SW105 SW_DPST_x2, SW106 SW_DPST_x2, SW107 SW_DPST_x2, SW108 SW_DPST_x2, SW11 SW_DPST_x2, SW12 SW_DPST_x2, SW13 SW_DPST_x2, SW14 SW_DPST_x2, SW15 SW_DPST_x2, SW16 SW_DPST_x2, SW17 SW_DPST_x2, SW18 SW_DPST_x2, SW19 SW_DPST_x2, SW2 SW_DPST_x2, SW20 SW_DPST_x2, SW21 SW_DPST_x2, SW22 SW_DPST_x2, SW23 SW_DPST_x2, SW24 SW_DPST_x2, SW25 SW_DPST_x2, SW26 SW_DPST_x2, SW27 SW_DPST_x2, SW28 SW_DPST_x2, SW29 SW_DPST_x2, SW3 SW_DPST_x2, SW30 SW_DPST_x2, SW31 SW_DPST_x2, SW32 SW_DPST_x2, SW33 SW_DPST_x2, SW34 SW_DPST_x2, SW35 SW_DPST_x2, SW36 SW_DPST_x2, SW37 SW_DPST_x2, SW38 SW_DPST_x2, SW39 SW_DPST_x2, SW4 SW_DPST_x2, SW40 SW_DPST_x2, SW41 SW_DPST_x2, SW42 SW_DPST_x2, SW43 SW_DPST_x2, SW44 SW_DPST_x2, SW45 SW_DPST_x2, SW46 SW_DPST_x2, SW47 SW_DPST_x2, SW48 SW_DPST_x2, SW49 SW_DPST_x2, SW5 SW_DPST_x2, SW50 SW_DPST_x2, SW51 SW_DPST_x2, SW52 SW_DPST_x2, SW53 SW_DPST_x2, SW54 SW_DPST_x2, SW55 SW_DPST_x2, SW56 SW_DPST_x2, SW57 SW_DPST_x2, SW58 SW_DPST_x2, SW59 SW_DPST_x2, SW6 SW_DPST_x2, SW60 SW_DPST_x2, SW61 SW_DPST_x2, SW62 SW_DPST_x2, SW63 SW_DPST_x2, SW64 SW_DPST_x2, SW65 SW_DPST_x2, SW66 SW_DPST_x2, SW67 SW_DPST_x2, SW68 SW_DPST_x2, SW69 SW_DPST_x2, SW7 SW_DPST_x2, SW70 SW_DPST_x2, SW71 SW_DPST_x2, SW72 SW_DPST_x2, SW73 SW_DPST_x2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

Commit message: hj
Parts:
- removed D1: 1N4148WT, Diode_SMD:D_SOD-523, symbol Diode:1N4148WT
- removed SW1, SW10, SW100, SW101, SW102, SW103, SW104, SW105, SW106, SW107, SW108, SW11, SW12, SW13, SW14, SW15, SW16, SW17, SW18, SW19, SW2, SW20, SW21, SW22, SW23, SW24, SW25, SW26, SW27, SW28, SW29, SW3, SW30, SW31, SW32, SW33, SW34, SW35, SW36, SW37, SW38, SW39, SW4, SW40, SW41, SW42, SW43, SW44, SW45, SW46, SW47, SW48, SW49, SW5, SW50, SW51, SW52, SW53, SW54, SW55, SW56, SW57, SW58, SW59, SW6, SW60, SW61, SW62, SW63, SW64, SW65, SW66, SW67, SW68, SW69, SW7, SW70, SW71, SW72, SW73, SW74, SW75, SW76, SW77, SW78, SW79, SW8, SW80, SW81, SW82, SW83, SW84, SW85, SW86, SW87, SW88, SW89, SW9, SW90, SW91, SW92, SW93, SW94, SW95, SW96, SW97, SW98, SW99: SW_DPST_x2, symbol Switch:SW_DPST_x2
- removed U1: Arduino_Micro, Arduino:Arduino_Micro, symbol Arduino:Arduino_Micro
- added A1: Arduino_Leonardo, Module:Arduino_UNO_R3, symbol MCU_Module:Arduino_Leonardo
- added D1, D10, D11, D12, D13, D14, D15, D16, D17, D18, D19, D2, D20, D21, D22, D23, D24, D25, D26, D27, D28, D29, D3, D30, D31, D32, D33, D34, D35, D36, D37, D38, D39, D4, D40, D41, D42, D43, D44, D45, D46, D47, D48, D49, D5, D50, D51, D52, D53, D54, D55, D56, D57, D58, D59, D6, D60, D61, D62, D63, D64, D65, D66, D67, D68, D69, D7, D70, D71, D72, D73, D74, D75, D76, D77, D78, D79, D8, D80, D81, D82, D83, D84, D85, D86, D87, D88, D89, D9, D90, D91, D92, D93, D94, D95, D96, D97, D98, D99: Diode, ScottoKeebs_Components:Diode_DO-35, symbol ScottoKeebs:Placeholder_Diode
- added S1, S10, S11, S12, S13, S14, S15, S16, S17, S18, S19, S2, S20, S21, S22, S23, S24, S25, S26, S27, S28, S29, S3, S30, S31, S32, S33, S34, S35, S36, S37, S38, S39, S4, S40, S41, S42, S43, S44, S45, S46, S47, S48, S49, S5, S50, S51, S52, S53, S54, S55, S56, S57, S58, S59, S6, S60, S61, S62, S63, S64, S65, S66, S67, S68, S69, S7, S70, S71, S72, S73, S74, S75, S76, S77, S78, S79, S8, S80, S81, S82, S83, S84, S85, S86, S87, S88, S89, S9, S90, S91, S92, S93, S94, S95, S96, S97, S98, S99: Keyswitch, ScottoKeebs_MX:MX_PCB_1.00u, symbol ScottoKeebs:Placeholder_Keyswitch
Connections:
- new net: D10.2 (A), S10.2
- new net: D64.2 (A), S64.2
- new net: D89.2 (A), S89.2
- new net: D15.2 (A), S15.2
- new net: D85.2 (A), S85.2
- new net: D44.2 (A), S44.2
- new net: D68.2 (A), S68.2
- new net: D90.2 (A), S90.2
- new net: D99.2 (A), S99.2
- new net: D35.2 (A), S35.2
- new net: D75.2 (A), S75.2
- new net: D25.2 (A), S25.2
- new net: D39.2 (A), S39.2
- new net: D55.2 (A), S55.2
- new net: D81.2 (A), S81.2
- new net: D74.2 (A), S74.2
- new net: D23.2 (A), S23.2
- new net: D72.2 (A), S72.2
- new net: D78.2 (A), S78.2
- new net: D32.2 (A), S32.2
- new net: D63.2 (A), S63.2
- new net: D1.2 (A), S1.2
- new net: D93.2 (A), S93.2
- new net: D51.2 (A), S51.2
- new net: D5.2 (A), S5.2
- new net: D2.2 (A), S2.2
- new net: D91.2 (A), S91.2
- new net: D92.2 (A), S92.2
- new net: D19.2 (A), S19.2
- new net: D84.2 (A), S84.2
- new net: D86.2 (A), S86.2
- new net: D80.2 (A), S80.2
- new net: D29.2 (A), S29.2
- new net: D43.2 (A), S43.2
- new net: D8.2 (A), S8.2
- new net: D12.2 (A), S12.2
- new net: D40.2 (A), S40.2
- new net: D11.2 (A), S11.2
- new net: D28.2 (A), S28.2
- new net: D22.2 (A), S22.2
- new net: D21.2 (A), S21.2
- new net: D69.2 (A), S69.2
- new net: D49.2 (A), S49.2
- new net: D94.2 (A), S94.2
- new net: D30.2 (A), S30.2
- new net: D97.2 (A), S97.2
- new net: D17.2 (A), S17.2
- new net: D56.2 (A), S56.2
- new net: D16.2 (A), S16.2
- new net: D53.2 (A), S53.2
- new net: D82.2 (A), S82.2
- new net: D37.2 (A), S37.2
- new net: D18.2 (A), S18.2
- new net: D9.2 (A), S9.2
- new net: D3.2 (A), S3.2
- new net: D87.2 (A), S87.2
- new net: D61.2 (A), S61.2
- new net: D59.2 (A), S59.2
- new net: D98.2 (A), S98.2
- new net: D70.2 (A), S70.2
- new net: D66.2 (A), S66.2
- new net: D31.2 (A), S31.2
- new net: D34.2 (A), S34.2
- new net: D54.2 (A), S54.2
- new net: D77.2 (A), S77.2
- new net: D88.2 (A), S88.2
- new net: D79.2 (A), S79.2
- new net: D52.2 (A), S52.2
- new net: D41.2 (A), S41.2
- new net: D71.2 (A), S71.2
- new net: D83.2 (A), S83.2
- new net: D42.2 (A), S42.2
- new net: D38.2 (A), S38.2
- new net: D4.2 (A), S4.2
- new net: D58.2 (A), S58.2
- new net: D60.2 (A), S60.2
- new net: D20.2 (A), S20.2
- new net: D27.2 (A), S27.2
- new net: D96.2 (A), S96.2
- new net: D48.2 (A), S48.2
- new net: D50.2 (A), S50.2
- new net: D33.2 (A), S33.2
- new net: D73.2 (A), S73.2
- new net: D62.2 (A), S62.2
- new net: D95.2 (A), S95.2
- new net: D36.2 (A), S36.2
- new net: D14.2 (A), S14.2
- new net: D65.2 (A), S65.2
- new net: D57.2 (A), S57.2
- new net: D67.2 (A), S67.2
- new net: D26.2 (A), S26.2
- new net: D47.2 (A), S47.2
- new net: D45.2 (A), S45.2
- new net: D24.2 (A), S24.2
- new net: D46.2 (A), S46.2
- new net: D13.2 (A), S13.2
- new net: D76.2 (A), S76.2
- new net: D6.2 (A), S6.2
- new net: D7.2 (A), S7.2
- new net Column 0: A1.25 (D10), S1.1, S11.1, S21.1, S31.1, S32.1, S33.1, S61.1, S62.1, S63.1, S64.1
- new net Column 1: A1.26 (D11), S12.1, S2.1, S22.1, S34.1, S35.1, S36.1, S65.1, S66.1, S67.1, S68.1
- new net Column 2: A1.27 (D12), S13.1, S23.1, S3.1, S37.1, S38.1, S39.1, S69.1, S70.1, S71.1, S72.1
- new net Column 3: A1.28 (D13), S14.1, S24.1, S4.1, S40.1, S41.1, S42.1, S73.1, S74.1, S75.1, S76.1
- new net Column 4: A1.9 (A0), S15.1, S25.1, S43.1, S44.1, S45.1, S5.1, S77.1, S78.1, S79.1, S80.1
- new net Column 5: A1.10 (A1), S16.1, S26.1, S46.1, S47.1, S48.1, S6.1, S81.1, S82.1, S83.1, S84.1
- new net Column 6: A1.11 (A2), S17.1, S27.1, S49.1, S50.1, S51.1, S7.1, S85.1, S86.1, S87.1, S88.1
- new net Column 7: A1.12 (A3), S18.1, S28.1, S52.1, S53.1, S54.1, S8.1, S89.1, S90.1, S91.1, S92.1
- new net Column 8: A1.13 (A4), S19.1, S29.1, S55.1, S56.1, S57.1, S9.1, S93.1, S94.1, S95.1, S96.1
- new net Column 9: A1.14 (A5), S10.1, S20.1, S30.1, S58.1, S59.1, S60.1, S97.1, S98.1, S99.1
- new net Row 0: A1.15 (D0/RX), D1.1 (K), D10.1 (K), D2.1 (K), D3.1 (K), D4.1 (K), D5.1 (K), D6.1 (K), D7.1 (K), D8.1 (K), D9.1 (K)
- new net Row 1: A1.16 (D1/TX), D11.1 (K), D12.1 (K), D13.1 (K), D14.1 (K), D15.1 (K), D16.1 (K), D17.1 (K), D18.1 (K), D19.1 (K), D20.1 (K)
- new net Row 2: A1.17 (D2/SDA), D21.1 (K), D22.1 (K), D23.1 (K), D24.1 (K), D25.1 (K), D26.1 (K), D27.1 (K), D28.1 (K), D29.1 (K), D30.1 (K)
- new net Row 3: A1.18 (D3/SCL), D31.1 (K), D34.1 (K), D37.1 (K), D40.1 (K), D43.1 (K), D46.1 (K), D49.1 (K), D52.1 (K), D55.1 (K), D58.1 (K)
- new net Row 4: A1.19 (D4), D32.1 (K), D35.1 (K), D38.1 (K), D41.1 (K), D44.1 (K), D47.1 (K), D50.1 (K), D53.1 (K), D56.1 (K), D59.1 (K)
- new net Row 5: A1.20 (D5), D33.1 (K), D36.1 (K), D39.1 (K), D42.1 (K), D45.1 (K), D48.1 (K), D51.1 (K), D54.1 (K), D57.1 (K), D60.1 (K)
- new net Row 6: A1.21 (D6), D61.1 (K), D65.1 (K), D69.1 (K), D73.1 (K), D77.1 (K), D81.1 (K), D85.1 (K), D89.1 (K), D93.1 (K), D97.1 (K)
- new net Row 7: A1.22 (D7), D62.1 (K), D66.1 (K), D70.1 (K), D74.1 (K), D78.1 (K), D82.1 (K), D86.1 (K), D90.1 (K), D94.1 (K), D98.1 (K)
- new net Row 8: A1.23 (D8), D63.1 (K), D67.1 (K), D71.1 (K), D75.1 (K), D79.1 (K), D83.1 (K), D87.1 (K), D91.1 (K), D95.1 (K), D99.1 (K)
- new net Row 9: A1.24 (D9), D64.1 (K), D68.1 (K), D72.1 (K), D76.1 (K), D80.1 (K), D84.1 (K), D88.1 (K), D92.1 (K), D96.1 (K)
