File: Chromatic/Chromatic.kicad_pcb (KiCad board)
At the start: 2 copper layers, 154 parts

Commit message: octave adjust
Parts:
- added R0: Resistor, Resistor_THT:R_Axial_DIN0204_L3.6mm_D1.6mm_P5.08mm_Horizontal, F.Cu at (9.50, 68.7)
- added R1: Resistor, Resistor_THT:R_Axial_DIN0204_L3.6mm_D1.6mm_P5.08mm_Horizontal, F.Cu at (28.5, 68.7)
- added R2: Resistor, Resistor_THT:R_Axial_DIN0204_L3.6mm_D1.6mm_P5.08mm_Horizontal, B.Cu at (47.5, 68.7)
- moved A1 25.8 mm to (51.1, -10.3)
- moved D_R0C0 11.7 mm to (9.66, 87.8)
- moved D_R0C1 11.7 mm to (9.66, 106.8)
- moved D_R0C13 11.7 mm to (9.66, 334.8)
- moved D_R0C15 11.7 mm to (9.66, 372.8)
- moved D_R0C16 11.7 mm to (9.66, 391.8)
- moved D_R1C0 11.7 mm to (28.7, 97.2)
- moved D_R1C1 11.7 mm to (28.9, 116.2)
- moved D_R1C16 11.7 mm to (28.7, 401.2)
- moved D_R1C2 11.7 mm to (28.9, 135.2)
- moved D_R1C3 11.7 mm to (28.7, 154.2)
- moved D_R1C4 11.7 mm to (28.9, 173.2)
- moved D_R1C5 11.7 mm to (28.9, 192.2)
- moved D_R1C6 11.7 mm to (28.7, 211.2)
- moved D_R1C7 11.7 mm to (28.9, 230.2)
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Connections:
- D_R0C0 pad 1: Row 0 -> Net-(D_R0C0-K)
- D_R0C1 pad 1: Row 0 -> Net-(D_R0C0-K)
- D_R0C10 pad 1: Row 0 -> Net-(D_R0C0-K)
- D_R0C11 pad 1: Row 0 -> Net-(D_R0C0-K)
- D_R0C12 pad 1: Row 0 -> Net-(D_R0C0-K)
- D_R0C13 pad 1: Row 0 -> Net-(D_R0C0-K)
- D_R0C14 pad 1: Row 0 -> Net-(D_R0C0-K)
- D_R0C15 pad 1: Row 0 -> Net-(D_R0C0-K)
- D_R0C16 pad 1: Row 0 -> Net-(D_R0C0-K)
- D_R0C2 pad 1: Row 0 -> Net-(D_R0C0-K)
- D_R0C3 pad 1: Row 0 -> Net-(D_R0C0-K)
- D_R0C4 pad 1: Row 0 -> Net-(D_R0C0-K)
- D_R0C5 pad 1: Row 0 -> Net-(D_R0C0-K)
- D_R0C6 pad 1: Row 0 -> Net-(D_R0C0-K)
- D_R0C7 pad 1: Row 0 -> Net-(D_R0C0-K)
- D_R0C8 pad 1: Row 0 -> Net-(D_R0C0-K)
- D_R0C9 pad 1: Row 0 -> Net-(D_R0C0-K)
- D_R1C0 pad 1: Row 1 -> Net-(D_R1C0-K)
- D_R1C1 pad 1: Row 1 -> Net-(D_R1C0-K)
- D_R1C10 pad 1: Row 1 -> Net-(D_R1C0-K)
- D_R1C11 pad 1: Row 1 -> Net-(D_R1C0-K)
- D_R1C12 pad 1: Row 1 -> Net-(D_R1C0-K)
- D_R1C13 pad 1: Row 1 -> Net-(D_R1C0-K)
- D_R1C14 pad 1: Row 1 -> Net-(D_R1C0-K)
- D_R1C15 pad 1: Row 1 -> Net-(D_R1C0-K)
- D_R1C16 pad 1: Row 1 -> Net-(D_R1C0-K)
- D_R1C2 pad 1: Row 1 -> Net-(D_R1C0-K)
- D_R1C3 pad 1: Row 1 -> Net-(D_R1C0-K)
- D_R1C4 pad 1: Row 1 -> Net-(D_R1C0-K)
- D_R1C5 pad 1: Row 1 -> Net-(D_R1C0-K)
- D_R1C6 pad 1: Row 1 -> Net-(D_R1C0-K)
- D_R1C7 pad 1: Row 1 -> Net-(D_R1C0-K)
- D_R1C8 pad 1: Row 1 -> Net-(D_R1C0-K)
- D_R1C9 pad 1: Row 1 -> Net-(D_R1C0-K)
- D_R2C0 pad 1: Row 2 -> Net-(D_R2C0-K)
- D_R2C1 pad 1: Row 2 -> Net-(D_R2C0-K)
- D_R2C10 pad 1: Row 2 -> Net-(D_R2C0-K)
- D_R2C11 pad 1: Row 2 -> Net-(D_R2C0-K)
- D_R2C12 pad 1: Row 2 -> Net-(D_R2C0-K)
- D_R2C13 pad 1: Row 2 -> Net-(D_R2C0-K)
- D_R2C14 pad 1: Row 2 -> Net-(D_R2C0-K)
- D_R2C15 pad 1: Row 2 -> Net-(D_R2C0-K)
- D_R2C16 pad 1: Row 2 -> Net-(D_R2C0-K)
- D_R2C2 pad 1: Row 2 -> Net-(D_R2C0-K)
- D_R2C3 pad 1: Row 2 -> Net-(D_R2C0-K)
- D_R2C4 pad 1: Row 2 -> Net-(D_R2C0-K)
- D_R2C5 pad 1: Row 2 -> Net-(D_R2C0-K)
- D_R2C6 pad 1: Row 2 -> Net-(D_R2C0-K)
- D_R2C7 pad 1: Row 2 -> Net-(D_R2C0-K)
- D_R2C8 pad 1: Row 2 -> Net-(D_R2C0-K)
- D_R2C9 pad 1: Row 2 -> Net-(D_R2C0-K)
Routing:
- net Row 1: track 345.2 -> 0.00 mm
- net Row 2: track 329.9 -> 1.33 mm
- net Row 0: track 330.3 -> 3.22 mm
- net Net-(D_R1C0-K): track 0.00 -> 323.6 mm
- net Net-(D_R2C0-K): track 0.00 -> 304.1 mm
- net Net-(D_R0C0-K): track 0.00 -> 304.0 mm
- net Column 0: track 128.8 -> 70.0 mm

Commit message: atualização
Parts:
- R0, R1: footprint Resistor_THT:R_Axial_DIN0204_L3.6mm_D1.6mm_P5.08mm_Horizontal -> Resistor_THT:R_Axial_DIN0309_L9.0mm_D3.2mm_P12.70mm_Horizontal
- R2: footprint Resistor_THT:R_Axial_DIN0204_L3.6mm_D1.6mm_P5.08mm_Horizontal -> Resistor_THT:R_Axial_DIN0309_L9.0mm_D3.2mm_P12.70mm_Horizontal; moved to F.Cu
- moved D_R1C16 413.4 mm to (385.6, 192.6), turned to 90 degrees
- moved SW_1_R1C16 408.9 mm to (394.1, 190.7), turned to 90 degrees
- moved SW_4_R1C16 408.4 mm to (403.6, 133.7), turned to 90 degrees
- moved D_R0C16 408.3 mm to (376.1, 211.5), turned to 90 degrees
- moved SW_0_R0C16 404.2 mm to (384.6, 209.7), turned to 90 degrees
- moved SW_3_R0C16 397.9 mm to (394.1, 152.7), turned to 90 degrees
- moved D_R2C16 394.2 mm to (375.9, 173.5), turned to 90 degrees
- moved SW_5_R2C16 393.9 mm to (394.1, 114.7), turned to 90 degrees
- moved SW_2_R2C16 389.4 mm to (384.6, 171.7), turned to 90 degrees
- moved D_R1C15 387.6 mm to (366.6, 192.8), turned to 90 degrees
- moved SW_1_R1C15 383.1 mm to (375.1, 190.7), turned to 90 degrees
- moved D_R0C15 383.0 mm to (357.1, 211.5), turned to 90 degrees
- moved SW_4_R1C15 381.6 mm to (384.6, 133.7), turned to 90 degrees
- moved SW_0_R0C15 379.1 mm to (365.6, 209.7), turned to 90 degrees
- moved SW_3_R0C15 371.3 mm to (375.1, 152.7), turned to 90 degrees
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Connections:
- A1 pad 10: Column 12 -> Column 15
- A1 pad 11: Column 13 -> Column 14
- A1 pad 12: Column 14 -> Column 13
- A1 pad 13: Column 15 -> Column 12
- A1 pad 14: Column 16 -> Column 11
- A1 pad 16: Column 0 -> Row 1
- A1 pad 17: Column 1 -> Row 2
- A1 pad 18: Column 10 -> Column 0
- A1 pad 19: Column 9 -> Column 1
- A1 pad 20: Column 8 -> Column 2
- A1 pad 21: Column 7 -> Column 3
- A1 pad 22: Column 6 -> Column 4
- A1 pad 24: Column 4 -> Column 6
- A1 pad 25: Column 3 -> Column 7
- A1 pad 26: Column 2 -> Column 8
- A1 pad 27: Row 1 -> Column 9
- A1 pad 28: Row 2 -> Column 10
- A1 pad 9: Column 11 -> Column 16
- R1 pad 1: Row 0 -> Row 1
- R2 pad 1: Row 0 -> Row 2
Routing:
- net Column 16: track 0.00 -> 549.3 mm
- net Column 15: track 0.00 -> 530.1 mm
- net Column 14: track 0.00 -> 511.3 mm
- net Column 13: track 0.00 -> 492.6 mm
- net Column 12: track 0.00 -> 472.9 mm
- net Column 11: track 0.00 -> 453.8 mm
- net Column 10: track 0.00 -> 375.9 mm
- net Column 9: track 0.00 -> 357.7 mm
- net Column 8: track 0.00 -> 339.2 mm
- net Column 7: track 0.00 -> 321.6 mm
- net Column 6: track 0.00 -> 302.8 mm
- net Column 5: track 0.00 -> 284.9 mm
- net Column 4: track 0.00 -> 268.2 mm
- net Column 3: track 0.00 -> 249.0 mm
- net Column 2: track 0.00 -> 230.7 mm
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Other:
- board outline added: 404.7 x 141.9 mm
