File: kicad_project/Chromatic.kicad_pcb (KiCad board)
At the start: 2 copper layers, 404.7 x 141.9 mm, 157 parts

Commit message: pc utf
Parts:
- SW_3_R0C16: footprint ScottoKeebs_Hotswap:Hotswap_MX_1.00u -> ScottoKeebs_Scotto:MX_Hotswap_1.00u; moved to B.Cu
- moved D_R0C13 83.3 mm to (343.0, 131.8)
- moved D_R0C14 83.3 mm to (362.0, 131.6)
- moved D_R0C15 83.3 mm to (381.0, 131.8)
- moved D_R0C16 83.3 mm to (400.0, 131.8)
- moved D_R1C12 83.3 mm to (333.5, 113.0)
- moved D_R1C13 83.3 mm to (352.5, 113.0)
- moved D_R1C14 83.3 mm to (371.5, 113.0)
- moved D_R1C15 83.3 mm to (390.5, 113.0)
- moved D_R2C13 83.3 mm to (342.8, 93.9)
- moved D_R2C14 83.3 mm to (361.8, 93.9)
- moved D_R2C15 83.3 mm to (380.8, 94.2)
- moved D_R2C16 83.3 mm to (399.8, 93.7)
- moved SW_0_R0C12 83.3 mm to (332.5, 129.9)
- moved SW_0_R0C13 83.3 mm to (351.5, 129.9)
- moved SW_0_R0C14 83.3 mm to (370.5, 129.9)
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Connections:
- D_R0C12 pad 1: Net-(D_R0C0-K) -> Net-(D_R0C12-K)
- D_R0C13 pad 1: Net-(D_R0C0-K) -> Net-(D_R0C12-K)
- D_R0C14 pad 1: Net-(D_R0C0-K) -> Net-(D_R0C12-K)
- D_R0C15 pad 1: Net-(D_R0C0-K) -> Net-(D_R0C12-K)
- D_R0C16 pad 1: Net-(D_R0C0-K) -> Net-(D_R0C12-K)
- D_R1C12 pad 1: Net-(D_R1C0-K) -> Net-(D_R1C12-K)
- D_R1C13 pad 1: Net-(D_R1C0-K) -> Net-(D_R1C12-K)
- D_R1C14 pad 1: Net-(D_R1C0-K) -> Net-(D_R1C12-K)
- D_R1C15 pad 1: Net-(D_R1C0-K) -> Net-(D_R1C12-K)
- D_R1C16 pad 1: Net-(D_R1C0-K) -> Net-(D_R1C12-K)
- D_R2C12 pad 1: Net-(D_R2C0-K) -> unconnected-(D_R2C12-K-Pad1)
- D_R2C13 pad 1: Net-(D_R2C0-K) -> Net-(D_R2C13-K)
- D_R2C14 pad 1: Net-(D_R2C0-K) -> Net-(D_R2C13-K)
- D_R2C15 pad 1: Net-(D_R2C0-K) -> Net-(D_R2C13-K)
- D_R2C16 pad 1: Net-(D_R2C0-K) -> Net-(D_R2C13-K)
- R0 pad 2: Net-(D_R0C0-K) -> Net-(D_R0C12-K)
- R1 pad 2: Net-(D_R1C0-K) -> Net-(D_R1C12-K)
- R2 pad 2: Net-(D_R2C0-K) -> Net-(D_R2C13-K)
- SW_0_R0C12 pad 1: Column 12 -> Net-(SW_0_R0C12-Pad1)
- SW_0_R0C13 pad 1: Column 13 -> Net-(SW_0_R0C13-Pad1)
- SW_0_R0C14 pad 1: Column 14 -> Net-(SW_0_R0C14-Pad1)
- SW_0_R0C15 pad 1: Column 15 -> Net-(SW_0_R0C15-Pad1)
- SW_0_R0C16 pad 1: Column 16 -> Net-(SW_0_R0C16-Pad1)
- SW_1_R1C12 pad 1: Column 12 -> Net-(SW_0_R0C12-Pad1)
- SW_1_R1C13 pad 1: Column 13 -> Net-(SW_0_R0C13-Pad1)
- SW_1_R1C14 pad 1: Column 14 -> Net-(SW_0_R0C14-Pad1)
- SW_1_R1C15 pad 1: Column 15 -> Net-(SW_0_R0C15-Pad1)
- SW_1_R1C16 pad 1: Column 16 -> Net-(SW_0_R0C16-Pad1)
- SW_2_R2C12 pad 1: Column 12 -> Net-(SW_0_R0C12-Pad1)
- SW_2_R2C13 pad 1: Column 13 -> Net-(SW_0_R0C13-Pad1)
- SW_2_R2C14 pad 1: Column 14 -> Net-(SW_0_R0C14-Pad1)
- SW_2_R2C15 pad 1: Column 15 -> Net-(SW_0_R0C15-Pad1)
- SW_2_R2C16 pad 1: Column 16 -> Net-(SW_0_R0C16-Pad1)
- SW_3_R0C12 pad 1: Column 12 -> Net-(SW_0_R0C12-Pad1)
- SW_3_R0C13 pad 1: Column 13 -> Net-(SW_0_R0C13-Pad1)
- SW_3_R0C14 pad 1: Column 14 -> Net-(SW_0_R0C14-Pad1)
- SW_3_R0C15 pad 1: Column 15 -> Net-(SW_0_R0C15-Pad1)
- SW_3_R0C16 pad 1: Column 16 -> Net-(SW_0_R0C16-Pad1)
- SW_4_R1C12 pad 1: Column 12 -> Net-(SW_0_R0C12-Pad1)
- SW_4_R1C13 pad 1: Column 13 -> Net-(SW_0_R0C13-Pad1)
- SW_4_R1C14 pad 1: Column 14 -> Net-(SW_0_R0C14-Pad1)
- SW_4_R1C15 pad 1: Column 15 -> Net-(SW_0_R0C15-Pad1)
- SW_4_R1C16 pad 1: Column 16 -> Net-(SW_0_R0C16-Pad1)
- SW_5_R2C12 pad 1: Column 12 -> Net-(SW_0_R0C12-Pad1)
- SW_5_R2C13 pad 1: Column 13 -> Net-(SW_0_R0C13-Pad1)
- SW_5_R2C14 pad 1: Column 14 -> Net-(SW_0_R0C14-Pad1)
- SW_5_R2C15 pad 1: Column 15 -> Net-(SW_0_R0C15-Pad1)
- SW_5_R2C16 pad 1: Column 16 -> Net-(SW_0_R0C16-Pad1)
Routing:
- net Column 12: track 472.9 -> 317.3 mm
- net Net-(SW_0_R0C13-Pad1): track 0.00 -> 144.6 mm
- net Column 13: track 492.6 -> 348.1 mm
- net Column 16: track 549.3 -> 404.9 mm
- net Net-(SW_0_R0C16-Pad1): track 0.00 -> 144.4 mm
- net Column 14: track 511.3 -> 366.9 mm
- net Net-(SW_0_R0C14-Pad1): track 0.00 -> 144.4 mm
- net Net-(SW_0_R0C15-Pad1): track 0.00 -> 144.0 mm
- net Column 15: track 530.1 -> 386.0 mm
- net Net-(SW_0_R0C12-Pad1): track 0.00 -> 138.3 mm
- net Net-(D_R2C0-K): track 384.1 -> 269.0 mm
- net Net-(D_R1C12-K): track 0.00 -> 115.1 mm
- net Net-(D_R1C0-K): track 390.6 -> 275.5 mm
- net Net-(D_R0C0-K): track 384.0 -> 291.9 mm
- net Net-(D_R0C12-K): track 0.00 -> 92.1 mm
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Other:
- board size 404.7 x 141.9 mm -> 298 x 141.9 mm

Commit message: arrumadas as bibliotecas
Parts:
- SW_0_R0C0, SW_0_R0C1, SW_0_R0C10, SW_0_R0C11, SW_0_R0C12, SW_0_R0C13, SW_0_R0C14, SW_0_R0C15, SW_0_R0C16, SW_0_R0C2, SW_0_R0C3, SW_0_R0C4, SW_0_R0C5, SW_0_R0C6, SW_0_R0C7, SW_0_R0C8, SW_0_R0C9, SW_1_R1C0, SW_1_R1C1, SW_1_R1C10, SW_1_R1C11, SW_1_R1C12, SW_1_R1C13, SW_1_R1C14, SW_1_R1C15, SW_1_R1C16, SW_1_R1C2, SW_1_R1C3, SW_1_R1C4, SW_1_R1C5, SW_1_R1C6, SW_1_R1C7, SW_1_R1C8, SW_1_R1C9, SW_2_R2C0, SW_2_R2C1, SW_2_R2C10, SW_2_R2C11, SW_2_R2C12, SW_2_R2C13, SW_2_R2C14, SW_2_R2C15, SW_2_R2C16, SW_2_R2C2, SW_2_R2C3, SW_2_R2C4, SW_2_R2C5, SW_2_R2C6, SW_2_R2C7, SW_2_R2C8, SW_2_R2C9, SW_3_R0C0, SW_3_R0C1, SW_3_R0C10, SW_3_R0C11, SW_3_R0C12, SW_3_R0C13, SW_3_R0C14, SW_3_R0C15, SW_3_R0C2, SW_3_R0C3, SW_3_R0C4, SW_3_R0C5, SW_3_R0C6, SW_3_R0C7, SW_3_R0C8, SW_3_R0C9, SW_4_R1C0, SW_4_R1C1, SW_4_R1C10, SW_4_R1C11, SW_4_R1C12, SW_4_R1C13, SW_4_R1C14, SW_4_R1C15, SW_4_R1C16, SW_4_R1C2, SW_4_R1C3, SW_4_R1C4, SW_4_R1C5, SW_4_R1C6, SW_4_R1C7, SW_4_R1C8, SW_4_R1C9, SW_5_R2C0, SW_5_R2C1, SW_5_R2C10, SW_5_R2C11, SW_5_R2C12, SW_5_R2C13, SW_5_R2C14, SW_5_R2C15, SW_5_R2C16, SW_5_R2C2, SW_5_R2C3, SW_5_R2C4, SW_5_R2C5, SW_5_R2C6, SW_5_R2C7, SW_5_R2C8, SW_5_R2C9: footprint ScottoKeebs_Hotswap:Hotswap_MX_1.00u -> ScottoKeebs_MX:MX_PCB_1.00u
- SW_3_R0C16: footprint ScottoKeebs_Scotto:MX_Hotswap_1.00u -> ScottoKeebs_MX:MX_PCB_1.00u

Commit message: commit
Parts:
- removed A1: Arduino_Leonardo, Module:Arduino_UNO_R3
- added A3: Arduino_Leonardo_Shield, arduino-library:Arduino_Leonardo_Shield, F.Cu at (2.65, 7.03)
- added J1: J1, Connector_PinHeader_2.54mm:PinHeader_1x08_P2.54mm_Vertical, F.Cu at (283.5, 1.84)
- added J2: J2, Connector_PinHeader_2.54mm:PinHeader_1x08_P2.54mm_Vertical, F.Cu at (322.5, 2.10)
- moved D_R0C12 36.7 mm to (324.3, 131.6)
Connections:
- D_R0C0 pad 1: Net-(D_R0C0-K) -> D_R0C11
- D_R0C1 pad 1: Net-(D_R0C0-K) -> D_R0C11
- D_R0C10 pad 1: Net-(D_R0C0-K) -> D_R0C11
- D_R0C11 pad 1: Net-(D_R0C0-K) -> D_R0C11
- D_R0C2 pad 1: Net-(D_R0C0-K) -> D_R0C11
- D_R0C3 pad 1: Net-(D_R0C0-K) -> D_R0C11
- D_R0C4 pad 1: Net-(D_R0C0-K) -> D_R0C11
- D_R0C5 pad 1: Net-(D_R0C0-K) -> D_R0C11
- D_R0C6 pad 1: Net-(D_R0C0-K) -> D_R0C11
- D_R0C7 pad 1: Net-(D_R0C0-K) -> D_R0C11
- D_R0C8 pad 1: Net-(D_R0C0-K) -> D_R0C11
- D_R0C9 pad 1: Net-(D_R0C0-K) -> D_R0C11
- D_R1C0 pad 1: Net-(D_R1C0-K) -> D_R1C11
- D_R1C1 pad 1: Net-(D_R1C0-K) -> D_R1C11
- D_R1C10 pad 1: Net-(D_R1C0-K) -> D_R1C11
- D_R1C11 pad 1: Net-(D_R1C0-K) -> D_R1C11
- D_R1C2 pad 1: Net-(D_R1C0-K) -> D_R1C11
- D_R1C3 pad 1: Net-(D_R1C0-K) -> D_R1C11
- D_R1C4 pad 1: Net-(D_R1C0-K) -> D_R1C11
- D_R1C5 pad 1: Net-(D_R1C0-K) -> D_R1C11
- D_R1C6 pad 1: Net-(D_R1C0-K) -> D_R1C11
- D_R1C7 pad 1: Net-(D_R1C0-K) -> D_R1C11
- D_R1C8 pad 1: Net-(D_R1C0-K) -> D_R1C11
- D_R1C9 pad 1: Net-(D_R1C0-K) -> D_R1C11
- D_R2C0 pad 1: Net-(D_R2C0-K) -> D_R2C11
- D_R2C1 pad 1: Net-(D_R2C0-K) -> D_R2C11
- D_R2C10 pad 1: Net-(D_R2C0-K) -> D_R2C11
- D_R2C11 pad 1: Net-(D_R2C0-K) -> D_R2C11
- D_R2C12 pad 1: unconnected-(D_R2C12-K-Pad1) -> Net-(D_R2C12-K)
- D_R2C2 pad 1: Net-(D_R2C0-K) -> D_R2C11
- D_R2C3 pad 1: Net-(D_R2C0-K) -> D_R2C11
- D_R2C4 pad 1: Net-(D_R2C0-K) -> D_R2C11
- D_R2C5 pad 1: Net-(D_R2C0-K) -> D_R2C11
- D_R2C6 pad 1: Net-(D_R2C0-K) -> D_R2C11
- D_R2C7 pad 1: Net-(D_R2C0-K) -> D_R2C11
- D_R2C8 pad 1: Net-(D_R2C0-K) -> D_R2C11
- D_R2C9 pad 1: Net-(D_R2C0-K) -> D_R2C11
- R0 pad 2: Net-(D_R0C12-K) -> D_R0C11
- R1 pad 2: Net-(D_R1C12-K) -> D_R1C11
- R2 pad 2: Net-(D_R2C13-K) -> D_R2C11
Routing:
- net (no net): track 0.00 -> 574.0 mm
- net D_R0C11: track 0.00 -> 389.3 mm
- net D_R1C11: track 0.00 -> 383.0 mm
- net Row 2: track 19.5 -> 395.4 mm
- net Column 10: track 375.9 -> 0.00 mm
- net D_R2C11: track 0.00 -> 359.0 mm
- net Net-(D_R0C0-K): track 291.9 -> 0.00 mm
- net Net-(D_R1C0-K): track 275.5 -> 0.00 mm
- net Net-(D_R2C0-K): track 269.0 -> 0.00 mm
- net Column 9: track 357.7 -> 194.0 mm
- net Column 0: track 194.0 -> 357.7 mm
- net Net-(J2-Pin_4): track 144.6 -> 0.00 mm
- net Net-(J2-Pin_3): track 144.4 -> 0.00 mm
- net Net-(J2-Pin_2): track 144.0 -> 0.00 mm
- net Net-(J2-Pin_5): track 138.3 -> 0.00 mm
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
Commit message: separados grupos
Parts:
- D_R0C0, D_R0C1, D_R0C10, D_R0C11, D_R0C12, D_R0C13, D_R0C14, D_R0C15, D_R0C16, D_R0C2, D_R0C3, D_R0C4, D_R0C5, D_R0C6, D_R0C7, D_R0C8, D_R0C9, D_R1C0, D_R1C1, D_R1C10, D_R1C11, D_R1C12, D_R1C13, D_R1C14, D_R1C15, D_R1C16, D_R1C2, D_R1C3, D_R1C4, D_R1C5, D_R1C6, D_R1C7, D_R1C8, D_R1C9, D_R2C0, D_R2C1, D_R2C10, D_R2C11, D_R2C12, D_R2C13, D_R2C14, D_R2C15, D_R2C16, D_R2C2, D_R2C3, D_R2C4, D_R2C5, D_R2C6, D_R2C7, D_R2C8, D_R2C9: moved to F.Cu
- SW_0_R0C0, SW_0_R0C1, SW_0_R0C10, SW_0_R0C11, SW_0_R0C12, SW_0_R0C13, SW_0_R0C14, SW_0_R0C15, SW_0_R0C16, SW_0_R0C2, SW_0_R0C3, SW_0_R0C4, SW_0_R0C5, SW_0_R0C6, SW_0_R0C7, SW_0_R0C8, SW_0_R0C9, SW_1_R1C0, SW_1_R1C1, SW_1_R1C10, SW_1_R1C11, SW_1_R1C12, SW_1_R1C13, SW_1_R1C14, SW_1_R1C15, SW_1_R1C16, SW_1_R1C2, SW_1_R1C3, SW_1_R1C4, SW_1_R1C5, SW_1_R1C6, SW_1_R1C7, SW_1_R1C8, SW_1_R1C9, SW_2_R2C0, SW_2_R2C1, SW_2_R2C10, SW_2_R2C11, SW_2_R2C12, SW_2_R2C13, SW_2_R2C14, SW_2_R2C15, SW_2_R2C16, SW_2_R2C2, SW_2_R2C3, SW_2_R2C4, SW_2_R2C5, SW_2_R2C6, SW_2_R2C7, SW_2_R2C8, SW_2_R2C9, SW_3_R0C0, SW_3_R0C1, SW_3_R0C10, SW_3_R0C11, SW_3_R0C12, SW_3_R0C13, SW_3_R0C14, SW_3_R0C15, SW_3_R0C2, SW_3_R0C3, SW_3_R0C4, SW_3_R0C5, SW_3_R0C6, SW_3_R0C7, SW_3_R0C8, SW_3_R0C9, SW_4_R1C0, SW_4_R1C1, SW_4_R1C10, SW_4_R1C11, SW_4_R1C12, SW_4_R1C13, SW_4_R1C14, SW_4_R1C15, SW_4_R1C16, SW_4_R1C2, SW_4_R1C3, SW_4_R1C4, SW_4_R1C5, SW_4_R1C6, SW_4_R1C7, SW_4_R1C8, SW_4_R1C9, SW_5_R2C0, SW_5_R2C1, SW_5_R2C10, SW_5_R2C11, SW_5_R2C12, SW_5_R2C13, SW_5_R2C14, SW_5_R2C15, SW_5_R2C16, SW_5_R2C2, SW_5_R2C3, SW_5_R2C4, SW_5_R2C5, SW_5_R2C6, SW_5_R2C7, SW_5_R2C8, SW_5_R2C9: footprint ScottoKeebs_MX:MX_PCB_1.00u -> ScottoKeebs_Scotto:MX_Hotswap_1.00u
- SW_3_R0C16: footprint ScottoKeebs_MX:MX_PCB_1.00u -> ScottoKeebs_Scotto:MX_Hotswap_1.00u; moved to F.Cu
- moved SW_4_R1C11 489.1 mm to (-76.0, 323.0), turned to 180 degrees
- moved SW_1_R1C11 465.9 mm to (-132.9, 313.5), turned to 180 degrees
- moved SW_0_R0C11 463.0 mm to (-151.9, 304.0), turned to 180 degrees
- moved D_R1C11 454.0 mm to (-131.6, 308.7), turned to 180 degrees
- moved D_R0C11 451.5 mm to (-150.6, 299.2), turned to 180 degrees
- moved SW_3_R0C11 451.0 mm to (-94.9, 313.5), turned to 180 degrees
- moved SW_2_R2C11 444.8 mm to (-113.9, 304.0), turned to 180 degrees
- moved SW_5_R2C11 442.3 mm to (-57.0, 313.5), turned to 180 degrees
- moved SW_1_R1C10 440.6 mm to (-132.9, 294.5), turned to 180 degrees
- moved SW_0_R0C10 438.4 mm to (-151.9, 285.0), turned to 180 degrees
- moved SW_4_R1C10 432.7 mm to (-76.0, 304.0), turned to 180 degrees
- moved D_R2C11 432.5 mm to (-112.3, 299.2), turned to 180 degrees
- moved J1 431.9 mm to (-23.2, 306.0), turned to -90 degrees
- moved D_R1C10 428.8 mm to (-131.6, 289.7), turned to 180 degrees
- moved D_R0C10 426.9 mm to (-150.6, 280.2), turned to 180 degrees
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Routing:
- net (no net): track 574.0 -> 0.00 mm
- net Column 11: track 455.7 -> 0.00 mm
- net Row 2: track 395.4 -> 0.00 mm
- net D_R0C11: track 389.3 -> 0.00 mm
- net D_R1C11: track 383.0 -> 0.00 mm
- net D_R2C11: track 359.0 -> 0.00 mm
- net Column 0: track 357.7 -> 0.00 mm
- net Column 1: track 339.2 -> 0.00 mm
- net Column 2: track 321.6 -> 0.00 mm
- net Column 3: track 302.8 -> 0.00 mm
- net Column 16: track 301.9 -> 0.00 mm
- net Column 12: track 301.5 -> 0.00 mm
- net Column 15: track 301.5 -> 0.00 mm
- net Column 14: track 301.5 -> 0.00 mm
- net Column 13: track 301.5 -> 0.00 mm
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Other:
- board outline removed
