File: kicad_project/Chromatic.kicad_pcb (KiCad board)
At the start: 2 copper layers, 159 parts, among them J1 J1, J2 J2

Commit message: layout
Parts:
- D_R0C0, D_R0C1, D_R0C10, D_R0C11, D_R0C2, D_R0C3, D_R0C4, D_R0C5, D_R0C6, D_R0C7, D_R0C8, D_R0C9, D_R1C0, D_R1C1, D_R1C10, D_R1C11, D_R1C2, D_R1C3, D_R1C4, D_R1C5, D_R1C6, D_R1C7, D_R1C8, D_R1C9, D_R2C0, D_R2C1, D_R2C10, D_R2C11, D_R2C2, D_R2C3, D_R2C4, D_R2C5, D_R2C6, D_R2C7, D_R2C8, D_R2C9: moved to B.Cu
- SW_0_R0C0, SW_0_R0C1, SW_0_R0C10, SW_0_R0C11, SW_0_R0C2, SW_0_R0C3, SW_0_R0C4, SW_0_R0C5, SW_0_R0C6, SW_0_R0C7, SW_0_R0C8, SW_0_R0C9, SW_1_R1C0, SW_1_R1C1, SW_1_R1C10, SW_1_R1C11, SW_1_R1C2, SW_1_R1C3, SW_1_R1C4, SW_1_R1C5, SW_1_R1C6, SW_1_R1C7, SW_1_R1C8, SW_1_R1C9, SW_2_R2C0, SW_2_R2C1, SW_2_R2C10, SW_2_R2C11, SW_2_R2C2, SW_2_R2C3, SW_2_R2C4, SW_2_R2C5, SW_2_R2C6, SW_2_R2C7, SW_2_R2C8, SW_2_R2C9, SW_3_R0C0, SW_3_R0C1, SW_3_R0C10, SW_3_R0C11, SW_3_R0C2, SW_3_R0C3, SW_3_R0C4, SW_3_R0C5, SW_3_R0C6, SW_3_R0C7, SW_3_R0C8, SW_3_R0C9, SW_4_R1C0, SW_4_R1C1, SW_4_R1C10, SW_4_R1C11, SW_4_R1C2, SW_4_R1C3, SW_4_R1C4, SW_4_R1C5, SW_4_R1C6, SW_4_R1C7, SW_4_R1C8, SW_4_R1C9, SW_5_R2C0, SW_5_R2C1, SW_5_R2C10, SW_5_R2C11, SW_5_R2C2, SW_5_R2C3, SW_5_R2C4, SW_5_R2C5, SW_5_R2C6, SW_5_R2C7, SW_5_R2C8, SW_5_R2C9: footprint ScottoKeebs_Scotto:MX_Hotswap_1.00u -> ScottoKeebs_Hotswap:Hotswap_MX_1.00u; moved to F.Cu
- SW_0_R0C12, SW_0_R0C13, SW_0_R0C14, SW_0_R0C15, SW_0_R0C16, SW_1_R1C12, SW_1_R1C13, SW_1_R1C14, SW_1_R1C15, SW_1_R1C16, SW_2_R2C12, SW_2_R2C13, SW_2_R2C14, SW_2_R2C15, SW_2_R2C16, SW_3_R0C12, SW_3_R0C13, SW_3_R0C14, SW_3_R0C15, SW_3_R0C16, SW_4_R1C12, SW_4_R1C13, SW_4_R1C14, SW_4_R1C15, SW_4_R1C16, SW_5_R2C12, SW_5_R2C13, SW_5_R2C14, SW_5_R2C15, SW_5_R2C16: footprint ScottoKeebs_Scotto:MX_Hotswap_1.00u -> ScottoKeebs_Hotswap:Hotswap_MX_1.00u
- moved D_R1C11 661.1 mm to (-473.1, 222.1)
- moved D_R1C10 658.4 mm to (-473.1, 203.1)
- moved D_R1C9 656.0 mm to (-473.1, 184.1)
- moved D_R0C0 652.8 mm to (-491.9, 3.56)
- moved D_R0C11 651.9 mm to (-491.9, 212.6)
- moved D_R0C1 651.1 mm to (-492.1, 22.6)
- moved D_R0C10 650.4 mm to (-492.1, 193.6)
- moved D_R0C2 649.5 mm to (-492.1, 41.6)
- moved D_R0C9 649.0 mm to (-492.1, 174.6)
- moved D_R2C11 648.4 mm to (-453.6, 212.6)
- moved D_R0C3 648.4 mm to (-492.1, 60.6)
- moved D_R0C8 648.0 mm to (-492.1, 155.6)
- moved D_R0C4 647.5 mm to (-492.1, 79.6)
- moved D_R0C7 647.3 mm to (-492.1, 136.6)
- moved D_R0C5 647.1 mm to (-492.1, 98.6)
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Routing:
- net Column 1: track 0.00 -> 114.3 mm
- net Column 0: track 0.00 -> 114.1 mm

Commit message: groups
Parts:
- moved D_R2C0 62.7 mm to (-514.7, -10.8), turned to 180 degrees
- moved D_R2C1 62.7 mm to (-514.7, 8.23), turned to 180 degrees
- moved D_R2C11 62.7 mm to (-514.6, 198.2), turned to 180 degrees
- moved D_R2C2 62.7 mm to (-514.7, 27.2), turned to 180 degrees
- moved D_R2C3 62.7 mm to (-514.7, 46.2), turned to 180 degrees
- moved D_R2C4 62.7 mm to (-514.7, 65.2), turned to 180 degrees
- moved D_R2C10 62.7 mm to (-514.5, 179.2), turned to 180 degrees
- moved D_R2C5 62.7 mm to (-514.5, 84.2), turned to 180 degrees
- moved D_R2C6 62.7 mm to (-514.5, 103.2), turned to 180 degrees
- moved D_R2C7 62.7 mm to (-514.5, 122.2), turned to 180 degrees
- moved D_R2C8 62.7 mm to (-514.5, 141.2), turned to 180 degrees
- moved D_R2C9 62.7 mm to (-514.5, 160.2), turned to 180 degrees
- moved D_R0C0 62.1 mm to (-552.2, -10.8), turned to 180 degrees
- moved D_R0C11 62.1 mm to (-552.2, 198.2), turned to 180 degrees
- moved D_R0C1 62.1 mm to (-552.5, 8.21), turned to 180 degrees
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Routing:
- net Column 1: track 114.3 -> 0.00 mm
- net Column 0: track 114.1 -> 0.00 mm

Commit message: COPPER LAYERS
Parts:
- moved D_R0C0 76.6 mm to (-475.8, -6.60)
- moved D_R0C11 76.6 mm to (-475.8, 202.4)
- moved D_R1C0 76.6 mm to (-456.8, 2.92)
- moved D_R1C1 76.6 mm to (-456.8, 21.9)
- moved D_R1C10 76.6 mm to (-456.8, 192.9)
- moved D_R1C11 76.6 mm to (-456.8, 211.9)
- moved D_R1C2 76.6 mm to (-456.8, 40.9)
- moved D_R1C3 76.6 mm to (-456.8, 59.9)
- moved D_R1C4 76.6 mm to (-456.8, 78.9)
- moved D_R1C5 76.6 mm to (-456.8, 97.9)
- moved D_R1C6 76.6 mm to (-456.8, 116.9)
- moved D_R1C7 76.6 mm to (-456.8, 135.9)
- moved D_R1C8 76.6 mm to (-456.8, 154.9)
- moved D_R1C9 76.6 mm to (-456.8, 173.9)
- moved D_R2C0 76.6 mm to (-438.3, -6.58)
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Routing:
- net D_R0C11: track 0.00 -> 244.1 mm
- net D_R1C11: track 0.00 -> 243.8 mm
- net D_R2C11: track 0.00 -> 243.2 mm
- net Column 6: track 0.00 -> 170.7 mm
- net Column 9: track 0.00 -> 170.0 mm
- net Column 11: track 0.00 -> 170.0 mm
- net Column 3: track 0.00 -> 169.5 mm
- net Column 7: track 0.00 -> 169.2 mm
- net Column 5: track 0.00 -> 169.0 mm
- net Column 2: track 0.00 -> 168.4 mm
- net Column 8: track 0.00 -> 167.0 mm
- net Column 10: track 0.00 -> 167.0 mm
- net Column 4: track 0.00 -> 166.8 mm
- net Column 1: track 0.00 -> 165.8 mm
- net Column 0: track 0.00 -> 164.4 mm
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