File: kicad_project/Chromatic.kicad_pcb (KiCad board)
At the start: 2 copper layers, 159 parts, among them J1 J1, J2 J2

Commit message: TROCADO ARDUINO POR ESP
Parts:
- removed A3: Arduino_Leonardo_Shield, Arduino:ARDUINO_A000066
- added U1: ESP32-S3, Module:XCVR_ESP32-S3-DEVKIT-LIPO, B.Cu at (143.1, 41.7)
- moved R1 1.50 mm to (68.0, 69.8)
Routing:
- net Column 11: track 497.2 -> 0.00 mm
- net Column 10: track 423.0 -> 0.00 mm
- net Column 9: track 398.3 -> 0.00 mm
- net Column 8: track 379.0 -> 0.00 mm
- net Column 7: track 360.8 -> 0.00 mm
- net D_R0C11: track 350.8 -> 0.00 mm
- net Column 6: track 344.5 -> 0.00 mm
- net D_R1C11: track 341.2 -> 0.00 mm
- net D_R2C11: track 330.2 -> 0.00 mm
- net Column 5: track 324.7 -> 0.00 mm
- net Column 16: track 299.8 -> 0.00 mm
- net Column 14: track 299.7 -> 0.00 mm
- net Column 13: track 299.6 -> 0.00 mm
- net Column 12: track 299.4 -> 0.00 mm
- net Column 15: track 299.4 -> 0.00 mm
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
Commit message: arrumado pcb e footprint
Parts:
- removed D_R0C14, D_R0C15, D_R0C16, D_R1C14, D_R1C15, D_R1C16, D_R2C14, D_R2C15, D_R2C16: ~, ScottoKeebs_Components:Diode_DO-35
- removed J1: J1, Connector_PinHeader_2.54mm:PinHeader_1x08_P2.54mm_Vertical
- removed J2: J2, Connector_PinHeader_2.54mm:PinHeader_1x08_P2.54mm_Vertical
- removed SW_0_R0C14, SW_0_R0C15, SW_0_R0C16, SW_1_R1C14, SW_1_R1C15, SW_1_R1C16, SW_2_R2C14, SW_2_R2C15, SW_2_R2C16, SW_3_R0C14, SW_3_R0C15, SW_3_R0C16, SW_4_R1C14, SW_4_R1C15, SW_4_R1C16, SW_5_R2C14, SW_5_R2C15, SW_5_R2C16: Keyswitch, ScottoKeebs_Hotswap:Hotswap_MX_1.00u
- removed U1: ESP32-S3, Module:XCVR_ESP32-S3-DEVKIT-LIPO
- added D_R2C17: ~, ScottoKeebs_Components:Diode_DO-35, F.Cu at (91.3, -36.9)
- added D_R2C18: ~, ScottoKeebs_Components:Diode_DO-35, F.Cu at (91.3, -33.3)
- added D_R2C19: ~, ScottoKeebs_Components:Diode_DO-35, F.Cu at (91.3, -29.8)
- added D_R2C20: ~, ScottoKeebs_Components:Diode_DO-35, F.Cu at (91.3, -26.2)
- added D_R2C21: ~, ScottoKeebs_Components:Diode_DO-35, F.Cu at (91.3, -22.7)
- added D_R2C22: ~, ScottoKeebs_Components:Diode_DO-35, F.Cu at (91.3, -19.1)
- added D_R2C23: ~, ScottoKeebs_Components:Diode_DO-35, F.Cu at (91.3, -15.6)
- added D_R2C24: ~, ScottoKeebs_Components:Diode_DO-35, F.Cu at (91.3, -12.0)
- added D_R2C25: ~, ScottoKeebs_Components:Diode_DO-35, F.Cu at (91.3, -8.47)
- added D_R2C26: ~, ScottoKeebs_Components:Diode_DO-35, F.Cu at (91.3, -4.92)
- added D_R2C27: ~, ScottoKeebs_Components:Diode_DO-35, F.Cu at (91.3, -1.37)
- added D_R2C28: ~, ScottoKeebs_Components:Diode_DO-35, F.Cu at (91.3, 2.18)
- added D_R2C29: ~, ScottoKeebs_Components:Diode_DO-35, F.Cu at (102.0, -36.9)
- added D_R2C30: ~, ScottoKeebs_Components:Diode_DO-35, F.Cu at (112.0, 39.2)
- added D_R2C31: ~, ScottoKeebs_Components:Diode_DO-35, F.Cu at (102.0, -29.8)
- added D_R2C32: ~, ScottoKeebs_Components:Diode_DO-35, F.Cu at (102.0, -26.2)
- added D_R2C33: ~, ScottoKeebs_Components:Diode_DO-35, F.Cu at (102.0, -22.7)
- added D_R2C34: ~, ScottoKeebs_Components:Diode_DO-35, F.Cu at (102.0, -19.1)
- added D_R2C35: ~, ScottoKeebs_Components:Diode_DO-35, F.Cu at (102.0, -15.6)
- added D_R2C36: ~, ScottoKeebs_Components:Diode_DO-35, F.Cu at (102.0, -12.0)
- added D_R2C37: ~, ScottoKeebs_Components:Diode_DO-35, F.Cu at (102.0, -8.47)
- added D_R2C38: ~, ScottoKeebs_Components:Diode_DO-35, F.Cu at (102.0, -4.92)
- added D_R2C39: ~, ScottoKeebs_Components:Diode_DO-35, F.Cu at (102.0, -1.37)
- added D_R2C40: ~, ScottoKeebs_Components:Diode_DO-35, F.Cu at (102.0, 2.18)
- added D_R2C41: ~, ScottoKeebs_Components:Diode_DO-35, F.Cu at (112.8, -36.9)
- added D_R2C42: ~, ScottoKeebs_Components:Diode_DO-35, F.Cu at (112.8, -33.3)
- added D_R2C43: ~, ScottoKeebs_Components:Diode_DO-35, F.Cu at (112.8, -29.8)
- added D_R2C44: ~, ScottoKeebs_Components:Diode_DO-35, F.Cu at (112.8, -26.2)
- added D_R2C45: ~, ScottoKeebs_Components:Diode_DO-35, F.Cu at (112.8, -22.7)
- added D_R2C46: ~, ScottoKeebs_Components:Diode_DO-35, F.Cu at (112.8, -19.1)
- added D_R2C47: ~, ScottoKeebs_Components:Diode_DO-35, F.Cu at (112.8, -15.6)
- added D_R2C48: ~, ScottoKeebs_Components:Diode_DO-35, F.Cu at (112.8, -12.0)
- added D_R2C49: ~, ScottoKeebs_Components:Diode_DO-35, F.Cu at (112.8, -8.47)
- added D_R2C50: ~, ScottoKeebs_Components:Diode_DO-35, F.Cu at (112.8, -4.92)
- added D_R2C51: ~, ScottoKeebs_Components:Diode_DO-35, F.Cu at (112.8, -1.37)
- added D_R2C52: ~, ScottoKeebs_Components:Diode_DO-35, F.Cu at (112.8, 2.18)
- added D_R2C53: ~, ScottoKeebs_Components:Diode_DO-35, F.Cu at (156.3, -9.93)
- added D_R2C54: ~, ScottoKeebs_Components:Diode_DO-35, F.Cu at (156.3, -6.38)
- added D_R2C55: ~, ScottoKeebs_Components:Diode_DO-35, F.Cu at (156.3, -2.83)
- added D_R2C56: ~, ScottoKeebs_Components:Diode_DO-35, F.Cu at (156.3, 0.72)
- added D_R2C57: ~, ScottoKeebs_Components:Diode_DO-35, F.Cu at (156.3, 4.28)
- added D_R2C58: ~, ScottoKeebs_Components:Diode_DO-35, F.Cu at (156.3, 7.83)
- added R3: Resistor, Resistor_THT:R_Axial_DIN0207_L6.3mm_D2.5mm_P7.62mm_Horizontal, F.Cu at (123.6, -36.6)
- added R4: Resistor, Resistor_THT:R_Axial_DIN0207_L6.3mm_D2.5mm_P7.62mm_Horizontal, F.Cu at (123.6, -32.6)
- added R5: Resistor, Resistor_THT:R_Axial_DIN0207_L6.3mm_D2.5mm_P7.62mm_Horizontal, F.Cu at (123.6, -28.5)
- added U2: ESP32-S3-DEVKITC-1-N8R8, RF_Module:ESP32-S3-DEVKITC-1-N8R8, F.Cu at (171.0, 161.5)
- moved SW_4_R1C12 102.8 mm to (95.0, 248.6)
- moved SW_4_R1C13 102.8 mm to (95.0, 267.6)
- moved D_R0C13 85.7 mm to (36.5, 266.3)
- moved D_R1C12 85.7 mm to (55.3, 256.8)
- moved D_R1C13 85.7 mm to (55.5, 275.8)
- moved D_R2C13 85.7 mm to (74.5, 266.3)
- moved D_R0C12 85.7 mm to (36.1, 248.3)
- moved D_R2C12 85.7 mm to (75.1, 248.3)
- moved SW_0_R0C12 85.7 mm to (19.0, 247.2)
- moved SW_2_R2C12 85.7 mm to (57.0, 247.2)
- moved SW_0_R0C13 85.7 mm to (19.0, 266.2)
- moved SW_1_R1C12 85.7 mm to (38.0, 256.7)
- moved SW_1_R1C13 85.7 mm to (38.0, 275.7)
- moved SW_2_R2C13 85.7 mm to (57.0, 266.2)
- moved SW_3_R0C12 85.7 mm to (76.0, 256.7)
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Connections:
- D_R0C0 pad 1: D_R0C11 -> Net-(D_R0C0-K)
- D_R0C1 pad 1: D_R0C11 -> Net-(D_R0C0-K)
- D_R0C10 pad 1: D_R0C11 -> Net-(D_R0C0-K)
- D_R0C11 pad 1: D_R0C11 -> Net-(D_R0C0-K)
- D_R0C12 pad 1: Net-(D_R0C12-K) -> Net-(D_R0C0-K)
- D_R0C13 pad 1: Net-(D_R0C12-K) -> Net-(D_R0C0-K)
- D_R0C2 pad 1: D_R0C11 -> Net-(D_R0C0-K)
- D_R0C3 pad 1: D_R0C11 -> Net-(D_R0C0-K)
- D_R0C4 pad 1: D_R0C11 -> Net-(D_R0C0-K)
- D_R0C5 pad 1: D_R0C11 -> Net-(D_R0C0-K)
- D_R0C6 pad 1: D_R0C11 -> Net-(D_R0C0-K)
- D_R0C7 pad 1: D_R0C11 -> Net-(D_R0C0-K)
- D_R0C8 pad 1: D_R0C11 -> Net-(D_R0C0-K)
- D_R0C9 pad 1: D_R0C11 -> Net-(D_R0C0-K)
- D_R1C0 pad 1: D_R1C11 -> Net-(D_R1C0-K)
- D_R1C1 pad 1: D_R1C11 -> Net-(D_R1C0-K)
- D_R1C10 pad 1: D_R1C11 -> Net-(D_R1C0-K)
- D_R1C11 pad 1: D_R1C11 -> Net-(D_R1C0-K)
- D_R1C12 pad 1: Net-(D_R1C12-K) -> Net-(D_R1C0-K)
- D_R1C13 pad 1: Net-(D_R1C12-K) -> Net-(D_R1C0-K)
- D_R1C2 pad 1: D_R1C11 -> Net-(D_R1C0-K)
- D_R1C3 pad 1: D_R1C11 -> Net-(D_R1C0-K)
- D_R1C4 pad 1: D_R1C11 -> Net-(D_R1C0-K)
- D_R1C5 pad 1: D_R1C11 -> Net-(D_R1C0-K)
- D_R1C6 pad 1: D_R1C11 -> Net-(D_R1C0-K)
- D_R1C7 pad 1: D_R1C11 -> Net-(D_R1C0-K)
- D_R1C8 pad 1: D_R1C11 -> Net-(D_R1C0-K)
- D_R1C9 pad 1: D_R1C11 -> Net-(D_R1C0-K)
- D_R2C0 pad 1: D_R2C11 -> Net-(D_R2C0-K)
- D_R2C1 pad 1: D_R2C11 -> Net-(D_R2C0-K)
- D_R2C10 pad 1: D_R2C11 -> Net-(D_R2C0-K)
- D_R2C11 pad 1: D_R2C11 -> Net-(D_R2C0-K)
- D_R2C12 pad 1: Net-(D_R2C12-K) -> Net-(D_R2C0-K)
- D_R2C13 pad 1: Net-(D_R2C12-K) -> Net-(D_R2C0-K)
- D_R2C2 pad 1: D_R2C11 -> Net-(D_R2C0-K)
- D_R2C3 pad 1: D_R2C11 -> Net-(D_R2C0-K)
- D_R2C4 pad 1: D_R2C11 -> Net-(D_R2C0-K)
- D_R2C5 pad 1: D_R2C11 -> Net-(D_R2C0-K)
- D_R2C6 pad 1: D_R2C11 -> Net-(D_R2C0-K)
- D_R2C7 pad 1: D_R2C11 -> Net-(D_R2C0-K)
- D_R2C8 pad 1: D_R2C11 -> Net-(D_R2C0-K)
- D_R2C9 pad 1: D_R2C11 -> Net-(D_R2C0-K)
- R0 pad 2: D_R0C11 -> Net-(D_R0C0-K)
- R1 pad 1: Row 1 -> Row 2
- R1 pad 2: D_R1C11 -> Net-(D_R1C0-K)
- R2 pad 1: Row 2 -> Row 4
- R2 pad 2: D_R2C11 -> Net-(D_R2C0-K)
- SW_0_R0C12 pad 1: Net-(J2-Pin_1) -> Column 9
- SW_0_R0C13 pad 1: Net-(J2-Pin_2) -> Column 10
- SW_1_R1C12 pad 1: Net-(J2-Pin_1) -> Column 9
- SW_1_R1C13 pad 1: Net-(J2-Pin_2) -> Column 10
- SW_2_R2C12 pad 1: Net-(J2-Pin_1) -> Column 9
- SW_2_R2C13 pad 1: Net-(J2-Pin_2) -> Column 10
- SW_3_R0C0 pad 2: Net-(D_R0C0-A) -> Net-(D_R2C41-A)
- SW_3_R0C1 pad 2: Net-(D_R0C1-A) -> Net-(D_R2C42-A)
- SW_3_R0C10 pad 2: Net-(D_R0C10-A) -> Net-(D_R2C51-A)
- SW_3_R0C11 pad 2: Net-(D_R0C11-A) -> Net-(D_R2C52-A)
- SW_3_R0C12 pad 1: Net-(J2-Pin_1) -> Column 9
- SW_3_R0C12 pad 2: Net-(D_R0C12-A) -> Net-(D_R2C53-A)
- SW_3_R0C13 pad 1: Net-(J2-Pin_2) -> Column 10
- SW_3_R0C13 pad 2: Net-(D_R0C13-A) -> Net-(D_R2C56-A)
- SW_3_R0C2 pad 2: Net-(D_R0C2-A) -> Net-(D_R2C43-A)
- SW_3_R0C3 pad 2: Net-(D_R0C3-A) -> Net-(D_R2C44-A)
- SW_3_R0C4 pad 2: Net-(D_R0C4-A) -> Net-(D_R2C45-A)
- SW_3_R0C5 pad 2: Net-(D_R0C5-A) -> Net-(D_R2C46-A)
- SW_3_R0C6 pad 2: Net-(D_R0C6-A) -> Net-(D_R2C47-A)
- SW_3_R0C7 pad 2: Net-(D_R0C7-A) -> Net-(D_R2C48-A)
- SW_3_R0C8 pad 2: Net-(D_R0C8-A) -> Net-(D_R2C49-A)
- SW_3_R0C9 pad 2: Net-(D_R0C9-A) -> Net-(D_R2C50-A)
- SW_4_R1C0 pad 2: Net-(D_R1C0-A) -> Net-(D_R2C29-A)
- SW_4_R1C1 pad 2: Net-(D_R1C1-A) -> Net-(D_R2C30-A)
- SW_4_R1C10 pad 2: Net-(D_R1C10-A) -> Net-(D_R2C39-A)
- SW_4_R1C11 pad 2: Net-(D_R1C11-A) -> Net-(D_R2C40-A)
- SW_4_R1C12 pad 1: Net-(J2-Pin_1) -> Column 9
- SW_4_R1C12 pad 2: Net-(D_R1C12-A) -> Net-(D_R2C54-A)
- SW_4_R1C13 pad 1: Net-(J2-Pin_2) -> Column 10
- SW_4_R1C13 pad 2: Net-(D_R1C13-A) -> Net-(D_R2C57-A)
- SW_4_R1C2 pad 2: Net-(D_R1C2-A) -> Net-(D_R2C31-A)
- SW_4_R1C3 pad 2: Net-(D_R1C3-A) -> Net-(D_R2C32-A)
- SW_4_R1C4 pad 2: Net-(D_R1C4-A) -> Net-(D_R2C33-A)
- SW_4_R1C5 pad 2: Net-(D_R1C5-A) -> Net-(D_R2C34-A)
- SW_4_R1C6 pad 2: Net-(D_R1C6-A) -> Net-(D_R2C35-A)
- SW_4_R1C7 pad 2: Net-(D_R1C7-A) -> Net-(D_R2C36-A)
- SW_4_R1C8 pad 2: Net-(D_R1C8-A) -> Net-(D_R2C37-A)
- SW_4_R1C9 pad 2: Net-(D_R1C9-A) -> Net-(D_R2C38-A)
- SW_5_R2C0 pad 2: Net-(D_R2C0-A) -> Net-(D_R2C17-A)
- SW_5_R2C1 pad 2: Net-(D_R2C1-A) -> Net-(D_R2C18-A)
- SW_5_R2C10 pad 2: Net-(D_R2C10-A) -> Net-(D_R2C27-A)
- SW_5_R2C11 pad 2: Net-(D_R2C11-A) -> Net-(D_R2C28-A)
- SW_5_R2C12 pad 1: Net-(J2-Pin_1) -> Column 9
- SW_5_R2C12 pad 2: Net-(D_R2C12-A) -> Net-(D_R2C55-A)
- SW_5_R2C13 pad 1: Net-(J2-Pin_2) -> Column 10
- SW_5_R2C13 pad 2: Net-(D_R2C13-A) -> Net-(D_R2C58-A)
- SW_5_R2C2 pad 2: Net-(D_R2C2-A) -> Net-(D_R2C19-A)
- SW_5_R2C3 pad 2: Net-(D_R2C3-A) -> Net-(D_R2C20-A)
- SW_5_R2C4 pad 2: Net-(D_R2C4-A) -> Net-(D_R2C21-A)
- SW_5_R2C5 pad 2: Net-(D_R2C5-A) -> Net-(D_R2C22-A)
- SW_5_R2C6 pad 2: Net-(D_R2C6-A) -> Net-(D_R2C23-A)
- SW_5_R2C7 pad 2: Net-(D_R2C7-A) -> Net-(D_R2C24-A)
- SW_5_R2C8 pad 2: Net-(D_R2C8-A) -> Net-(D_R2C25-A)
- SW_5_R2C9 pad 2: Net-(D_R2C9-A) -> Net-(D_R2C26-A)
Routing:
- net Net-(D_R0C0-K): track 0.00 -> 288.8 mm
- net Net-(J2-Pin_1): track 258.9 -> 0.00 mm
- net Net-(J2-Pin_2): track 237.3 -> 0.00 mm
- net Column 0: track 0.00 -> 217.4 mm
- net Net-(J2-Pin_3): track 214.3 -> 0.00 mm
- net Net-(J2-Pin_4): track 211.1 -> 0.00 mm
- net Net-(J2-Pin_5): track 204.3 -> 0.00 mm
- net Net-(D_R0C12-K): track 193.1 -> 0.00 mm
- net Column 4: track 175.6 -> 0.00 mm
- net Column 2: track 174.2 -> 0.00 mm
- net Column 3: track 171.9 -> 0.00 mm
- net Net-(D_R1C12-K): track 164.5 -> 0.00 mm
- net Net-(D_R2C12-K): track 150.3 -> 0.00 mm
- net Net-(D_R2C12-A): track 79.6 -> 0.00 mm
- net Net-(D_R1C12-A): track 68.1 -> 0.00 mm
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